File: PCB Design/MCU_&_Power.kicad_sch (KiCad schematic)
At the start: 73 parts, among them SW10 SW_Push, SW11 SW_Push, SW12 SW_Push, SW13 SW_Push, SW14 SW_Push, SW3 RotaryEncoder_Switch, SW4 RotaryEncoder_Switch, SW5 RotaryEncoder_Switch, SW6 SW_Push, SW7 SW_Push, SW8 SW_Push, SW9 SW_Push

Commit message: Assign footprints
Parts:
- C25, C26, C27, C28, C29, C30, C31, C32, C33, C34, C35, C36, C37, C38, C39, C40, C41, C42, C43: footprint (none) -> Capacitor_SMD:C_0402_1005Metric
- H1: value MountingHole_Pad_MP -> MountingHole_Pad
- R25: value 100M -> 100m; footprint (none) -> Resistor_SMD:R_1206_3216Metric
- R26, R27, R28, R29, R30, R31, R32, R33, R34, R35, R36, R37: footprint (none) -> Resistor_SMD:R_0402_1005Metric
- SW10, SW11, SW12, SW13, SW14, SW6, SW7, SW8, SW9: footprint (none) -> Kailh_PG1353_Hotswap:Kailh-PG1353-Hotswap-1U
- SW3, SW4, SW5: footprint (none) -> Rotary_Encoder:RotaryEncoder_Bourns_Vertical_PEC12R-3x17F-Sxxxx
Other:
- moved on the sheet: R25
Changed lines of the file:
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@@
 	)
 	(junction
-		(at 16.51 25.4)
-		(diameter 0)
-		(color 0 0 0 0)
-	)
-	(junction
 		(at 151.13 31.75)
 		(diameter 0)
@@
 	)
 	(junction
+		(at 48.26 25.4)
+		(diameter 0)
+		(color 0 0 0 0)
+	)
+	(junction
 		(at 92.71 137.16)
 		(diameter 0)
@@
 			)
 		)
-		(property "Footprint" ""
+		(property "Footprint" "Kailh_PG1353_Hotswap:Kailh-PG1353-Hotswap-1U"
 			(at 262.89 130.81 0)
 			(effects
@@
 			)
 		)
-		(property "Footprint" ""
+		(property "Footprint" "Rotary_Encoder:RotaryEncoder_Bourns_Vertical_PEC12R-3x17F-Sxxxx"
 			(at 59.69 92.964 0)
 			(effects
@@
 			)
 		)
-		(property "Footprint" ""
+		(property "Footprint" "Resistor_SMD:R_0402_1005Metric"
 			(at 91.44 128.27 0)
 			(effects
@@
 			)
 		)
-		(property "Footprint" ""
+		(property "Footprint" "Kailh_PG1353_Hotswap:Kailh-PG1353-Hotswap-1U"
 			(at 262.89 83.82 0)
 			(effects
@@
 			)
 		)
-		(property "Footprint" ""
+		(property "Footprint" "Resistor_SMD:R_0402_1005Metric"
 			(at 72.39 167.64 0)
 			(effects
@@
 			)
 		)
-		(property "Value" "MountingHole_Pad_MP"
+		(property "Value" "MountingHole_Pad"
 			(at 139.7 99.0599 0)
 			(effects
@@
 			)
 		)
-		(property "Description" "Mounting Hole with connection as pad named MP"
+		(property "Description" "Mounting Hole with connection"
 			(at 137.16 99.06 0)
 			(effects
@@
 			)
 		)
-		(property "Footprint" ""
+		(property "Footprint" "Kailh_PG1353_Hotswap:Kailh-PG1353-Hotswap-1U"
 			(at 201.93 83.82 0)
 			(effects
@@
 			)
 		)
-		(property "Footprint" ""
+		(property "Footprint" "Resistor_SMD:R_0402_1005Metric"
 			(at 91.44 172.72 0)
 			(effects
@@
 	(symbol
 		(lib_id "power:+5V")
-		(at 16.51 20.32 0)
+		(at 48.26 20.32 0)
 		(unit 1)
 		(exclude_from_sim no)
@@
 		(fields_autoplaced yes)
 		(property "Reference" "#PWR048"
-			(at 16.51 24.13 0)
+			(at 48.26 24.13 0)
 			(effects
 				(font
@@
 		)
 		(property "Value" "+5V"
-			(at 16.51 15.24 0)
+			(at 48.26 15.24 0)
 			(effects
 				(font
@@
 		)
 		(property "Footprint" ""
-			(at 16.51 20.32 0)
+			(at 48.26 20.32 0)
 			(effects
 				(font
@@
 		)
 		(property "Datasheet" ""
-			(at 16.51 20.32 0)
+			(at 48.26 20.32 0)
 			(effects
 				(font
@@
 		)
 		(property "Description" "Power symbol creates a global label with name \"+5V\""
-			(at 16.51 20.32 0)
+			(at 48.26 20.32 0)
 			(effects
 				(font
@@
 			)
 		)
-		(property "Footprint" ""
+		(property "Footprint" "Resistor_SMD:R_0402_1005Metric"
 			(at 87.63 137.16 0)
 			(effects
@@
 			)
 		)
-		(property "Footprint" ""
+		(property "Footprint" "Capacitor_SMD:C_0402_1005Metric"
 			(at 218.44 46.99 0)
 			(effects
@@
 			)
 		)
-		(property "Footprint" ""
+		(property "Footprint" "Capacitor_SMD:C_0402_1005Metric"
 			(at 99.06 187.96 0)
 			(effects
@@
 			)
 		)
-		(property "Footprint" ""
+		(property "Footprint" "Capacitor_SMD:C_0402_1005Metric"
 			(at 92.71 143.51 0)
 			(effects
@@
 			)
 		)
-		(property "Footprint" ""
+		(property "Footprint" "Capacitor_SMD:C_0402_1005Metric"
 			(at 133.35 46.99 0)
 			(effects
@@
 			)
 		)
-		(property "Footprint" ""
+		(property "Footprint" "Capacitor_SMD:C_0402_1005Metric"
 			(at 20.32 177.8 0)
 			(effects
@@
 			)
 		)
-		(property "Footprint" ""
+		(property "Footprint" "Capacitor_SMD:C_0402_1005Metric"
 			(at 92.71 97.79 0)
 			(effects
@@
 			)
 		)
-		(property "Footprint" ""
+		(property "Footprint" "Resistor_SMD:R_0402_1005Metric"
 			(at 81.28 123.19 0)
 			(effects
@@
 			)
 		)
-		(property "Footprint" ""
+		(property "Footprint" "Resistor_SMD:R_0402_1005Metric"
 			(at 72.39 123.19 0)
 			(effects
@@
 			)
 		)
-		(property "Footprint" ""
+		(property "Footprint" "Kailh_PG1353_Hotswap:Kailh-PG1353-Hotswap-1U"
 			(at 232.41 83.82 0)
 			(effects
@@
 			)
 		)
-		(property "Footprint" ""
+		(property "Footprint" "Capacitor_SMD:C_0402_1005Metric"
 			(at 99.06 97.79 0)
 			(effects
@@
 			)
 		)
-		(property "Footprint" ""
+		(property "Footprint" "Capacitor_SMD:C_0402_1005Metric"
 			(at 190.5 46.99 0)
 			(effects
@@
 			)
 		)
-		(property "Footprint" ""
+		(property "Footprint" "Kailh_PG1353_Hotswap:Kailh-PG1353-Hotswap-1U"
 			(at 201.93 130.81 0)
 			(effects
@@
 			)
 		)
-		(property "Footprint" ""
+		(property "Footprint" "Capacitor_SMD:C_0402_1005Metric"
 			(at 20.32 87.63 0)
 			(effects
@@
 			)
 		)
-		(property "Footprint" ""
+		(property "Footprint" "Kailh_PG1353_Hotswap:Kailh-PG1353-Hotswap-1U"
 			(at 262.89 109.22 0)
 			(effects
@@
 			)
 		)
-		(property "Footprint" ""
+		(property "Footprint" "Resistor_SMD:R_0402_1005Metric"
 			(at 87.63 91.44 0)
 			(effects
@@
 			)
 		)
-		(property "Footprint" ""
+		(property "Footprint" "Resistor_SMD:R_0402_1005Metric"
 			(at 87.63 181.61 0)
 			(effects
@@
 			)
 		)
-		(property "Footprint" ""
+		(property "Footprint" "Kailh_PG1353_Hotswap:Kailh-PG1353-Hotswap-1U"
 			(at 201.93 106.68 0)
 			(effects
@@
 			)
 		)
-		(property "Footprint" ""
+		(property "Footprint" "Capacitor_SMD:C_0402_1005Metric"
 			(at 16.51 29.21 0)
 			(effects
@@
 			)
 		)
-		(property "Footprint" ""
+		(property "Footprint" "Resistor_SMD:R_0402_1005Metric"
 			(at 81.28 167.64 0)
 			(effects
@@
 			)
 		)
-		(property "Footprint" ""
+		(property "Footprint" "Capacitor_SMD:C_0402_1005Metric"
 			(at 20.32 132.08 0)
 			(effects
@@
 			)
 		)
-		(property "Footprint" ""
+		(property "Footprint" "Resistor_SMD:R_0402_1005Metric"
 			(at 72.39 77.47 0)
 			(effects
@@
 			)
 		)
-		(property "Footprint" ""
+		(property "Footprint" "Kailh_PG1353_Hotswap:Kailh-PG1353-Hotswap-1U"
 			(at 232.41 130.81 0)
 			(effects
@@
 			)
 		)
-		(property "Footprint" ""
+		(property "Footprint" "Capacitor_SMD:C_0402_1005Metric"
 			(at 245.11 46.99 0)
 			(effects
@@
 			)
 		)
-		(property "Footprint" ""
+		(property "Footprint" "Capacitor_SMD:C_0402_1005Metric"
 			(at 48.26 46.99 0)
 			(effects
@@
 			)
 		)
-		(property "Footprint" ""
+		(property "Footprint" "Capacitor_SMD:C_0402_1005Metric"
 			(at 105.41 46.99 0)
 			(effects
@@
 			)
 		)
-		(property "Footprint" ""
+		(property "Footprint" "Capacitor_SMD:C_0402_1005Metric"
 			(at 77.47 46.99 0)
 			(effects
@@
 			)
 		)
-		(property "Footprint" ""
+		(property "Footprint" "Rotary_Encoder:RotaryEncoder_Bourns_Vertical_PEC12R-3x17F-Sxxxx"
 			(at 59.69 138.684 0)
 			(effects
@@
 			)
 		)
-		(property "Footprint" ""
+		(property "Footprint" "Resistor_SMD:R_0402_1005Metric"
 			(at 91.44 82.55 0)
 			(effects
@@
 			)
 		)
-		(property "Footprint" ""
+		(property "Footprint" "Capacitor_SMD:C_0402_1005Metric"
 			(at 273.05 46.99 0)
 			(effects
@@
 			)
 		)
-		(property "Footprint" ""
+		(property "Footprint" "Kailh_PG1353_Hotswap:Kailh-PG1353-Hotswap-1U"
 			(at 232.41 109.22 0)
 			(effects
@@
 			)
 		)
-		(property "Footprint" ""
+		(property "Footprint" "Rotary_Encoder:RotaryEncoder_Bourns_Vertical_PEC12R-3x17F-Sxxxx"
 			(at 59.69 183.134 0)
 			(effects
@@
 	(symbol
 		(lib_id "Device:R_Small")
-		(at 16.51 22.86 180)
+		(at 48.26 22.86 180)
 		(unit 1)
 		(exclude_from_sim no)
@@
 		(fields_autoplaced yes)
 		(property "Reference" "R25"
-			(at 19.05 21.5899 0)
+			(at 50.8 21.5899 0)
 			(effects
 				(font
@@
 			)
 		)
-		(property "Value" "100M"
-			(at 19.05 24.1299 0)
+		(property "Value" "100m"
+			(at 50.8 24.1299 0)
 			(effects
 				(font
@@
 			)
 		)
-		(property "Footprint" ""
-			(at 16.51 22.86 0)
+		(property "Footprint" "Resistor_SMD:R_1206_3216Metric"
+			(at 48.26 22.86 0)
 			(effects
 				(font
@@
 		)
 		(property "Datasheet" "~"
-			(at 16.51 22.86 0)
+			(at 48.26 22.86 0)
 			(effects
 				(font
@@
 		)
 		(property "Description" "Resistor, small symbol"
-			(at 16.51 22.86 0)
+			(at 48.26 22.86 0)
 			(effects
 				(font
@@
 			)
 		)
-		(property "Footprint" ""
+		(property "Footprint" "Capacitor_SMD:C_0402_1005Metric"
 			(at 162.56 46.99 0)
 			(effects
@@
 			)
 		)
-		(property "Footprint" ""
+		(property "Footprint" "Capacitor_SMD:C_0402_1005Metric"
 			(at 99.06 143.51 0)
 			(effects
@@
 			)
 		)
-		(property "Footprint" ""
+		(property "Footprint" "Resistor_SMD:R_0402_1005Metric"
 			(at 81.28 77.47 0)
 			(effects
@@
 			)
 		)
-		(property "Footprint" ""
+		(property "Footprint" "Capacitor_SMD:C_0402_1005Metric"
 			(at 92.71 187.96 0)
 			(effects

Commit message: More footprints.
Parts:
- H1, H2, H3, H4: footprint (none) -> MountingHole:MountingHole_2.5mm_Pad_TopBottom
- H5, H6, H7, H8: footprint (none) -> MountingHole:MountingHole_3.5mm_Pad_TopBottom
Other:
- title: (none) -> MacroPad
Changed lines of the file:
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@@
 	(generator_version "9.0")
 	(paper "A4")
+	(title_block
+		(title "MacroPad")
+		(date "2025-04-20")
+		(rev "A")
+	)
 	(text "KEYSWITCH LED LIGHTING"
 		(exclude_from_sim no)
@@
 			)
 		)
-		(property "Footprint" ""
+		(property "Footprint" "MountingHole:MountingHole_3.5mm_Pad_TopBottom"
 			(at 163.83 137.16 0)
 			(effects
@@
 			)
 		)
-		(property "Footprint" ""
+		(property "Footprint" "MountingHole:MountingHole_2.5mm_Pad_TopBottom"
 			(at 137.16 99.06 0)
 			(effects
@@
 			)
 		)
-		(property "Footprint" ""
+		(property "Footprint" "MountingHole:MountingHole_2.5mm_Pad_TopBottom"
 			(at 163.83 99.06 0)
 			(effects
@@
 			)
 		)
-		(property "Footprint" ""
+		(property "Footprint" "MountingHole:MountingHole_2.5mm_Pad_TopBottom"
 			(at 146.05 99.06 0)
 			(effects
@@
 			)
 		)
-		(property "Footprint" ""
+		(property "Footprint" "MountingHole:MountingHole_3.5mm_Pad_TopBottom"
 			(at 139.7 137.16 0)
 			(effects
@@
 			)
 		)
-		(property "Footprint" ""
+		(property "Footprint" "MountingHole:MountingHole_3.5mm_Pad_TopBottom"
 			(at 163.83 118.11 0)
 			(effects
@@
 			)
 		)
-		(property "Footprint" ""
+		(property "Footprint" "MountingHole:MountingHole_3.5mm_Pad_TopBottom"
 			(at 139.7 118.11 0)
 			(effects
@@
 			)
 		)
-		(property "Footprint" ""
+		(property "Footprint" "MountingHole:MountingHole_2.5mm_Pad_TopBottom"
 			(at 154.94 99.06 0)
 			(effects
